File: pcb/SNES JAMMA.sch (EAGLE design)
At the start: 10 parts, among them P1-JAMMA-A PLAYER 1 JAMMA, P2-JAMMA-A PLAYER 2 JAMMA

Commit message: v1.0 PCB and Schematics files
Parts:
- removed P1-JAMMA-A: PLAYER 1 JAMMA, con-amp:MTA05-100
- removed P1-JAMMA-B, P2-JAMMA-B: (no value), con-amp:MTA06-100
- removed P2-JAMMA-A: PLAYER 2 JAMMA, con-amp:MTA05-100
- added J1: 12V POWER, con-amp:MTA02-100
- added J2: (no value), con-amp:MTA03-100
- added JAMMA: 057-040-1, con-panduit:057-040-1
Connections:
- net P1-H-KICK renamed P1-BTN6
- net P1-L-KICK renamed P1-BTN4
- net P1-M-KICK renamed P1-BTN5
- net P2-H-KICK renamed P2-BTN6
- net P2-L-KICK renamed P2-BTN4
- net P2-M-KICK renamed P2-BTN5
- removed net P1-JAMMA-COIN: P1-JAMMA-B.5, PLAYER-1.D11/MOSI
- removed net P1-JAMMA-DOWN: P1-JAMMA-A.3, PLAYER-1.D4
- removed net P1-JAMMA-H-PUNCH: P1-JAMMA-B.3, PLAYER-1.D9
- removed net P1-JAMMA-L-PUNCH: P1-JAMMA-B.1, PLAYER-1.D7
- removed net P1-JAMMA-LEFT: P1-JAMMA-A.4, PLAYER-1.D5
- removed net P1-JAMMA-M-PUNCH: P1-JAMMA-B.2, PLAYER-1.D8
- removed net P1-JAMMA-RIGHT: P1-JAMMA-A.5, PLAYER-1.D6
- removed net P1-JAMMA-START: P1-JAMMA-B.4, PLAYER-1.D10
- removed net P1-JAMMA-UP: P1-JAMMA-A.2, PLAYER-1.D3
- removed net P2-JAMMA-COIN: P2-JAMMA-B.2, PLAYER-2.D11/MOSI
- removed net P2-JAMMA-DOWN: P2-JAMMA-A.3, PLAYER-2.D4
- removed net P2-JAMMA-H-PUNCH: P2-JAMMA-B.4, PLAYER-2.D9
- removed net P2-JAMMA-L-PUNCH: P2-JAMMA-B.6, PLAYER-2.D7
- removed net P2-JAMMA-LEFT: P2-JAMMA-A.2, PLAYER-2.D5
- removed net P2-JAMMA-M-PUNCH: P2-JAMMA-B.5, PLAYER-2.D8
- removed net P2-JAMMA-RIGHT: P2-JAMMA-A.1, PLAYER-2.D6
- removed net P2-JAMMA-START: P2-JAMMA-B.3, PLAYER-2.D10
- removed net P2-JAMMA-UP: P2-JAMMA-A.4, PLAYER-2.D3
- new net +12V: J1.2, J2.1
- new net N$6: PLAYER-1.D12/MISO
- new net P1-BTN1: JAMMA-27.S, PLAYER-1.D9
- new net P1-BTN2: JAMMA-29.S, PLAYER-1.D10
- new net P1-BTN3: JAMMA-31.S, PLAYER-1.D11/MOSI
- new net P1-COIN: JAMMA-15.S, PLAYER-1.D3
- new net P1-DOWN: JAMMA-21.S, PLAYER-1.D6
- new net P1-LEFT: JAMMA-23.S, PLAYER-1.D7
- new net P1-RIGHT: JAMMA-25.S, PLAYER-1.D8
- new net P1-START: JAMMA-17.S, PLAYER-1.D4
- new net P1-UP: JAMMA-19.S, PLAYER-1.D5
- new net P2-BTN1: JAMMA-28.S, PLAYER-2.D9
- new net P2-BTN2: JAMMA-30.S, PLAYER-2.D10
- new net P2-BTN3: JAMMA-32.S, PLAYER-2.D11/MOSI
- new net P2-COIN: JAMMA-16.S, PLAYER-2.D3
- new net P2-DOWN: JAMMA-22.S, PLAYER-2.D6
- new net P2-LEFT: JAMMA-24.S, PLAYER-2.D7
- new net P2-RIGHT: JAMMA-26.S, PLAYER-2.D8
- new net P2-START: JAMMA-18.S, PLAYER-2.D4
- new net P2-UP: JAMMA-20.S, PLAYER-2.D5
- net GND: now also J1.1, J2.2; no longer P1-JAMMA-B.6, P2-JAMMA-B.1
- net VCC: now also J2.3; no longer P1-JAMMA-A.1, P2-JAMMA-A.5
Other:
- moved on the sheet: CPS1-KICK, EZ-KICK, PLAYER-1, PLAYER-2, SFC-PLAYER-1, SFC-PLAYER-2

Commit message: Updating board design to v1.1 Adding ability for P1 Arduino to trigger "test" switch
Connections:
- removed net N$3: PLAYER-1.D2
- new net TEST: JAMMA-14.S, PLAYER-1.D2
Other:
- moved on the sheet: JAMMA-14
Changed lines of the file:
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@@
 <attribute name="NAME" x="55.118" y="133.604" size="1.524" layer="95" rot="R270"/>
 </instance>
-<instance part="JAMMA" gate="-14" x="55.88" y="111.76" smashed="yes" rot="R270">
-<attribute name="NAME" x="55.118" y="110.744" size="1.524" layer="95" rot="R270"/>
+<instance part="JAMMA" gate="-14" x="60.96" y="76.2" smashed="yes">
+<attribute name="NAME" x="61.976" y="75.438" size="1.524" layer="95"/>
 </instance>
 <instance part="JAMMA" gate="-15" x="60.96" y="73.66" smashed="yes">
@@
 </segment>
 </net>
-<net name="N$3" class="0">
+<net name="TEST" class="0">
 <segment>
 <pinref part="PLAYER-1" gate="MODUL" pin="D2"/>
-<wire x1="38.1" y1="76.2" x2="40.64" y2="76.2" width="0.1524" layer="91"/>
-</segment>
-</net>
+<pinref part="JAMMA" gate="-14" pin="S"/>
+<wire x1="38.1" y1="76.2" x2="55.88" y2="76.2" width="0.1524" layer="91"/>
+<label x="43.18" y="76.2" size="1.778" layer="95"/>
+</segment>
+</net>

Commit message: Correcting P1 TEST toggle incorrectly being wired to TILT instead P1 TEST is now properly TEST toggle Additionally, P2's is now wired into TILT so they're both available to be used!
Connections:
- removed net N$11: PLAYER-2.D2
- new net TILT: JAMMA-14.S, PLAYER-2.D2
- net TEST: now also JAMMA-13.S; no longer JAMMA-14.S
Other:
- moved on the sheet: JAMMA-13, JAMMA-14
Changed lines of the file:
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@@
 <attribute name="NAME" x="60.198" y="110.744" size="1.524" layer="95" rot="R270"/>
 </instance>
-<instance part="JAMMA" gate="-13" x="55.88" y="134.62" smashed="yes" rot="R270">
-<attribute name="NAME" x="55.118" y="133.604" size="1.524" layer="95" rot="R270"/>
-</instance>
-<instance part="JAMMA" gate="-14" x="60.96" y="76.2" smashed="yes">
+<instance part="JAMMA" gate="-13" x="60.96" y="76.2" smashed="yes">
 <attribute name="NAME" x="61.976" y="75.438" size="1.524" layer="95"/>
+</instance>
+<instance part="JAMMA" gate="-14" x="106.68" y="76.2" smashed="yes" rot="R180">
+<attribute name="NAME" x="105.664" y="76.962" size="1.524" layer="95" rot="R180"/>
 </instance>
 <instance part="JAMMA" gate="-15" x="60.96" y="73.66" smashed="yes">
@@
 </segment>
 </net>
-<net name="TEST" class="0">
-<segment>
-<pinref part="PLAYER-1" gate="MODUL" pin="D2"/>
-<pinref part="JAMMA" gate="-14" pin="S"/>
-<wire x1="38.1" y1="76.2" x2="55.88" y2="76.2" width="0.1524" layer="91"/>
-<label x="43.18" y="76.2" size="1.778" layer="95"/>
-</segment>
-</net>
 <net name="N$4" class="0">
 <segment>
@@
 </segment>
 </net>
-<net name="N$11" class="0">
+<net name="TILT" class="0">
 <segment>
 <pinref part="PLAYER-2" gate="MODUL" pin="D2"/>
-<wire x1="132.08" y1="76.2" x2="129.54" y2="76.2" width="0.1524" layer="91"/>
+<pinref part="JAMMA" gate="-14" pin="S"/>
+<wire x1="132.08" y1="76.2" x2="111.76" y2="76.2" width="0.1524" layer="91"/>
+<label x="114.3" y="76.2" size="1.778" layer="95"/>
 </segment>
 </net>
@@
 </segment>
 </net>
+<net name="TEST" class="0">
+<segment>
+<pinref part="PLAYER-1" gate="MODUL" pin="D2"/>
+<pinref part="JAMMA" gate="-13" pin="S"/>
+<wire x1="38.1" y1="76.2" x2="55.88" y2="76.2" width="0.1524" layer="91"/>
+<label x="43.18" y="76.2" size="1.778" layer="95"/>
+</segment>
+</net>
